File: KiCad-files/BrodBoostC2Rebuild.kicad_pcb (KiCad board)
At the start: 2 copper layers, 54 x 35 mm, 38 parts, among them J1 USB_C_Receptacle_USB2.0_16P, J2 5v Power Rail, J3 3V3 Power Rail, SW1 SW_SPDT, U1 LM66100DCK, U2 TPS22918DBV, U3 AP2114H-3.3TRG1

Commit message: Update parts
Parts:
- D2, D3, D4, D5, D6, D7: footprint LED_SMD:LED_0603_1608Metric_Pad1.05x0.95mm_HandSolder -> LED_SMD:LED_0805_2012Metric_Pad1.15x1.40mm_HandSolder
- F1: footprint Fuse:Fuse_0603_1608Metric_Pad1.05x0.95mm_HandSolder -> Fuse:Fuse_0805_2012Metric_Pad1.15x1.40mm_HandSolder
Routing:
- net GND: vias 12 -> 7

Commit message: Updated board
Parts:
- F1: value Polyfuse -> Fuse
- FB1: value FerriteBead -> Ferrite
- R1, R10, R2, R4, R5, R6, R7, R8, R9: value 5.1k -> 5k1Ω
- R3: value 100 -> 100Ω
- moved H2 1.30 mm to (96.6, 73.0)
- moved H1 0.81 mm to (50.6, 73.0)
- moved R1 0.06 mm to (81.3, 74.4)
Routing:
- net Net-(J1-CC2): track 12.7 -> 13.7 mm
- net GND: vias 7 -> 6
Other:
- board text added: "+"
- board text added: "-"

Commit message: Updated schematic
Parts:
- R10, R5, R7, R8, R9: value 5k1Ω -> 2.2kΩ
- R6: value 5k1Ω -> 1kΩ
Other:
- board text added: "https://github.com/domesticmouse/BrodBoost-C2-rebuild"
