File: KiCad-files/BrodBoostC2Rebuild.kicad_sch (KiCad schematic)
At the start: 35 parts, among them J1 USB_C_Receptacle_USB2.0_16P, J2 Conn_02x03_Odd_Even, J3 Conn_02x03_Odd_Even, SW1 SW_SPDT, U1 LM66100DCK, U2 TPS22918DBV, U3 AP2114H-3.3TRG1

Commit message: Add PCB
Parts:
- removed TP1: V_BUS Raw, TestPoint:TestPoint_Keystone_5000-5004_Miniature, symbol Connector:TestPoint
- removed TP2: GND, TestPoint:TestPoint_Keystone_5000-5004_Miniature, symbol Connector:TestPoint
- removed TP3: USB D+, TestPoint:TestPoint_Keystone_5000-5004_Miniature, symbol Connector:TestPoint
- removed TP4: USB D-, TestPoint:TestPoint_Keystone_5000-5004_Miniature, symbol Connector:TestPoint
- removed TP5: V_BUS Protected, TestPoint:TestPoint_Keystone_5000-5004_Miniature, symbol Connector:TestPoint
- removed TP6: 5V, TestPoint:TestPoint_Keystone_5000-5004_Miniature, symbol Connector:TestPoint
- removed TP7: 3V3, TestPoint:TestPoint_Keystone_5000-5004_Miniature, symbol Connector:TestPoint
- added D4: USB D-, LED_SMD:LED_0603_1608Metric_Pad1.05x0.95mm_HandSolder, symbol Device:LED
- added D5: USB D+, LED_SMD:LED_0603_1608Metric_Pad1.05x0.95mm_HandSolder, symbol Device:LED
- added D6: VBUS, LED_SMD:LED_0603_1608Metric_Pad1.05x0.95mm_HandSolder, symbol Device:LED
- added D7: VBUS Protected, LED_SMD:LED_0603_1608Metric_Pad1.05x0.95mm_HandSolder, symbol Device:LED
- added H1, H2: MountingHole_Pad, MountingHole:MountingHole_3.2mm_M3_Pad, symbol Mechanical:MountingHole_Pad
- added R10, R7, R8, R9: 5.1k, Resistor_SMD:R_0805_2012Metric_Pad1.20x1.40mm_HandSolder, symbol Device:R
- D2: value LED -> 5V; LCSC C965799 -> C84256
- D3: value LED -> 3V3; LCSC C965799 -> C84256
- FB1: footprint (none) -> BrodBoostFootprints:FerriteBead_0805_2012Metric_Pad1.20x1.40mm_HandSolder
- J1: footprint (none) -> Connector_USB:USB_C_Receptacle_XKB_U262-16XN-4BVC11
- J2: value Conn_02x03_Odd_Even -> 5v Power Rail
- J3: value Conn_02x03_Odd_Even -> 3V3 Power Rail
- SW1: footprint (none) -> Button_Switch_THT:SW_Slide_SPDT_Straight_CK_OS102011MS2Q
Connections:
- net GND: now also D4.1 (K), D5.1 (K), D6.1 (K), D7.1 (K), H1.1, H2.1
- net USB-D+: now also R8.1
- net USB-D-: now also R7.1
- net V_BUS: now also R9.1
- net V_BUS_Protected: now also R10.1
- new net: D6.2 (A), R9.2
- new net: D4.2 (A), R7.2
- new net: D7.2 (A), R10.2
- new net: D5.2 (A), R8.2
Other:
- moved on the sheet: C10, C5, C6, C7, C8, C9, D2, D3, J2, R5, R6, U3

Commit message: Update parts
Parts:
- D2, D3, D4, D5, D6, D7: footprint LED_SMD:LED_0603_1608Metric_Pad1.05x0.95mm_HandSolder -> LED_SMD:LED_0805_2012Metric_Pad1.15x1.40mm_HandSolder
- F1: footprint Fuse:Fuse_0603_1608Metric_Pad1.05x0.95mm_HandSolder -> Fuse:Fuse_0805_2012Metric_Pad1.15x1.40mm_HandSolder; LCSC C18203128 -> C22363531
- FB1: LCSC C85840 -> C76818
- SW1: LCSC (none) -> C2939725
Changed lines of the file:
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@@
 			)
 		)
-		(property "Footprint" "LED_SMD:LED_0603_1608Metric_Pad1.05x0.95mm_HandSolder"
+		(property "Footprint" "LED_SMD:LED_0805_2012Metric_Pad1.15x1.40mm_HandSolder"
 			(at 132.08 139.7 0)
 			(hide yes)
@@
 			)
 		)
+		(property "LCSC" "C2939725"
+			(at 184.15 50.8 0)
+			(hide yes)
+			(show_name no)
+			(do_not_autoplace no)
+			(effects
+				(font
+					(size 1.27 1.27)
+				)
+			)
+		)
 		(pin "2"
 		)
@@
 			)
 		)
-		(property "LCSC" "C85840"
+		(property "LCSC" "C76818"
 			(at 113.03 27.94 90)
 			(hide yes)
@@
 			)
 		)
-		(property "Footprint" "Fuse:Fuse_0603_1608Metric_Pad1.05x0.95mm_HandSolder"
+		(property "Footprint" "Fuse:Fuse_0805_2012Metric_Pad1.15x1.40mm_HandSolder"
 			(at 106.68 26.67 0)
 			(hide yes)
@@
 			)
 		)
-		(property "LCSC" "C18203128"
+		(property "LCSC" "C22363531"
 			(at 101.6 27.94 90)
 			(hide yes)
@@
 			)
 		)
-		(property "Footprint" "LED_SMD:LED_0603_1608Metric_Pad1.05x0.95mm_HandSolder"
+		(property "Footprint" "LED_SMD:LED_0805_2012Metric_Pad1.15x1.40mm_HandSolder"
 			(at 203.2 139.7 0)
 			(hide yes)
@@
 			)
 		)
-		(property "Footprint" "LED_SMD:LED_0603_1608Metric_Pad1.05x0.95mm_HandSolder"
+		(property "Footprint" "LED_SMD:LED_0805_2012Metric_Pad1.15x1.40mm_HandSolder"
 			(at 175.26 139.7 0)
 			(hide yes)
@@
 			)
 		)
-		(property "Footprint" "LED_SMD:LED_0603_1608Metric_Pad1.05x0.95mm_HandSolder"
+		(property "Footprint" "LED_SMD:LED_0805_2012Metric_Pad1.15x1.40mm_HandSolder"
 			(at 161.29 139.7 0)
 			(hide yes)
@@
 			)
 		)
-		(property "Footprint" "LED_SMD:LED_0603_1608Metric_Pad1.05x0.95mm_HandSolder"
+		(property "Footprint" "LED_SMD:LED_0805_2012Metric_Pad1.15x1.40mm_HandSolder"
 			(at 146.05 139.7 0)
 			(hide yes)
@@
 			)
 		)
-		(property "Footprint" "LED_SMD:LED_0603_1608Metric_Pad1.05x0.95mm_HandSolder"
+		(property "Footprint" "LED_SMD:LED_0805_2012Metric_Pad1.15x1.40mm_HandSolder"
 			(at 189.23 139.7 0)
 			(hide yes)

Commit message: Updated board
Parts:
- F1: value Polyfuse -> Fuse
- FB1: value FerriteBead -> Ferrite
- R1, R10, R2, R4, R5, R6, R7, R8, R9: value 5.1k -> 5k1Ω
- R3: value 100 -> 100Ω
Changed lines of the file:
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@@
 			)
 		)
-		(property "Value" "5.1k"
+		(property "Value" "5k1Ω"
 			(at 58.42 43.18 90)
 			(show_name no)
@@
 			)
 		)
-		(property "Value" "5.1k"
+		(property "Value" "5k1Ω"
 			(at 148.59 129.5399 0)
 			(show_name no)
@@
 			)
 		)
-		(property "Value" "5.1k"
+		(property "Value" "5k1Ω"
 			(at 134.62 129.5399 0)
 			(show_name no)
@@
 			)
 		)
-		(property "Value" "100"
+		(property "Value" "100Ω"
 			(at 240.03 35.56 90)
 			(show_name no)
@@
 			)
 		)
-		(property "Value" "5.1k"
+		(property "Value" "5k1Ω"
 			(at 191.77 129.5399 0)
 			(show_name no)
@@
 			)
 		)
-		(property "Value" "FerriteBead"
+		(property "Value" "Ferrite"
 			(at 112.9792 22.86 90)
 			(show_name no)
@@
 			)
 		)
-		(property "Value" "5.1k"
+		(property "Value" "5k1Ω"
 			(at 163.83 129.5399 0)
 			(show_name no)
@@
 			)
 		)
-		(property "Value" "Polyfuse"
+		(property "Value" "Fuse"
 			(at 101.6 24.13 90)
 			(show_name no)
@@
 			)
 		)
-		(property "Value" "5.1k"
+		(property "Value" "5k1Ω"
 			(at 58.42 33.02 90)
 			(show_name no)
@@
 			)
 		)
-		(property "Value" "5.1k"
+		(property "Value" "5k1Ω"
 			(at 205.74 129.5399 0)
 			(show_name no)
@@
 			)
 		)
-		(property "Value" "5.1k"
+		(property "Value" "5k1Ω"
 			(at 176.53 39.3699 0)
 			(show_name no)
@@
 			)
 		)
-		(property "Value" "5.1k"
+		(property "Value" "5k1Ω"
 			(at 177.8 129.5399 0)
 			(show_name no)

Commit message: Updated schematic
Parts:
- R10, R5, R7, R8, R9: value 5k1Ω -> 2.2kΩ
- R6: value 5k1Ω -> 1kΩ
Changed lines of the file:
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@@
 			)
 		)
-		(property "Value" "5k1Ω"
+		(property "Value" "2.2kΩ"
 			(at 148.59 129.5399 0)
 			(show_name no)
@@
 			)
 		)
-		(property "Value" "5k1Ω"
+		(property "Value" "1kΩ"
 			(at 134.62 129.5399 0)
 			(show_name no)
@@
 			)
 		)
-		(property "Value" "5k1Ω"
+		(property "Value" "2.2kΩ"
 			(at 191.77 129.5399 0)
 			(show_name no)
@@
 			)
 		)
-		(property "Value" "5k1Ω"
+		(property "Value" "2.2kΩ"
 			(at 163.83 129.5399 0)
 			(show_name no)
@@
 			)
 		)
-		(property "Value" "5k1Ω"
+		(property "Value" "2.2kΩ"
 			(at 205.74 129.5399 0)
 			(show_name no)
@@
 			)
 		)
-		(property "Value" "5k1Ω"
+		(property "Value" "2.2kΩ"
 			(at 177.8 129.5399 0)
 			(show_name no)
